Commit message: [main] sync updates 01/14/2025

File: concepts/simulator/urdf_utils/urdf_prototype.urdf (robot description, URDF)
Before this commit: robot _name, 1 links, 0 joints
Links:
- removed link _name
- added link object, mass 1.0; collision mesh filename=_prototype.obj scale=1 1 1; visual mesh filename=_prototype.obj scale=1 1 1
